File: kicad/RadioSens.kicad_pcb (KiCad board)
At the start: 2 copper layers, 62.6 x 42.7 mm, 200 parts, among them J1 Spacer M2, J2 Spacer M2, J3 Spacer M2, J4 Spacer M2, J5 Spacer M2, J6 Spacer M2

Commit message: Add docs; Update values of components according to PCB
Parts:
- C26, C27: value 22u/50V -> 47u/50V
- C38: value 4.7u/25V -> 4.7u/6.3V
Changed lines of the file:
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@@
     (descr "DFN, 6 Pin (https://www.silabs.com/documents/public/data-sheets/Si7020-A20.pdf), generated with kicad-footprint-generator ipc_noLead_generator.py")
     (tags "DFN NoLead")
+    (property "Assembly" "")
+    (property "MNP" "")
     (property "Sheetfile" "iic_connector.kicad_sch")
     (property "Sheetname" "IIC Connector")
@@
       (effects (font (size 1 1) (thickness 0.15)))
     )
-    (fp_text value "22u/50V" (at 0 5.2 90) (layer "F.Fab")
+    (fp_text value "47u/50V" (at 0 5.2 90) (layer "F.Fab")
       (effects (font (size 1 1) (thickness 0.15)))
     )
@@
       (effects (font (size 1 1) (thickness 0.15)))
     )
-    (fp_text value "22u/50V" (at 0 5.2 90) (layer "F.Fab")
+    (fp_text value "47u/50V" (at 0 5.2 90) (layer "F.Fab")
       (effects (font (size 1 1) (thickness 0.15)))
     )
@@
       (effects (font (size 1 1) (thickness 0.15)))
     )
-    (fp_text value "4.7u/25V" (at 0 1.43 90) (layer "F.Fab")
+    (fp_text value "4.7u/6.3V" (at 0 1.43 90) (layer "F.Fab")
       (effects (font (size 1 1) (thickness 0.15)))
     )
@@
     (descr "Resistor SMD 0603 (1608 Metric), square (rectangular) end terminal, IPC_7351 nominal, (Body size source: IPC-SM-782 page 72, https://www.pcb-3d.com/wordpress/wp-content/uploads/ipc-sm-782a_amendment_1_and_2.pdf), generated with kicad-footprint-generator")
     (tags "resistor")
-    (property "Assembly" "")
+    (property "Assembly" "DNP")
     (property "Case/Package" "0603")
     (property "Part Number" "")
@@
     (descr "SOP, 8 Pin (http://www.macronix.com/Lists/Datasheet/Attachments/7534/MX25R3235F,%20Wide%20Range,%2032Mb,%20v1.6.pdf#page=79), generated with kicad-footprint-generator ipc_gullwing_generator.py")
     (tags "SOP SO")
-    (property "Assembly" "DNP")
+    (property "Assembly" "")
     (property "Link" "https://www.rcscomponents.kiev.ua/product/24lc64t-i-sn_14769.html")
     (property "Sheetfile" "iic_connector.kicad_sch")
